Commit message: chore: arm and panel removed entirely from the repository

File: src/rover/rover_description/urdf/rover.urdf.xacro (robot description, xacro)
@@ -7,7 +7,4 @@
   <xacro:include filename="$(find rover_description)/urdf/macros/stereo_camera.xacro"/>
   <xacro:include filename="$(find rover_description)/urdf/macros/lidar.xacro"/>
-  <xacro:if value="$(arg mount_arm)">
-    <xacro:include filename="$(find arm_description)/urdf/arm_macro.xacro"/>
-  </xacro:if>
   <!-- ===================== MATERIALS ===================== -->
   <material name="blue_body">
@@ -132,11 +129,3 @@
   <xacro:stop_button_accessory suffix="l" y_sign="1"/>
   <xacro:stop_button_accessory suffix="r" y_sign="-1"/>
-  <!-- ===================== ARM (OPTIONAL) ===================== -->
-  <!-- Placeholder mount pose; update once the real MR_ARM_ATT attachment
-       point from CAD is known. -->
-  <xacro:if value="$(arg mount_arm)">
-    <xacro:indomitus_arm parent_link="main_body_link">
-      <origin xyz="0.2 0 0.1" rpy="0 0 0"/>
-    </xacro:indomitus_arm>
-  </xacro:if>
 </robot>

File: src/rover/rover_description/urdf/rover.xacro (robot description, xacro)
@@ -23,6 +23,4 @@
   <xacro:arg name="stereo_camera_simulate_depth" default="false"/>
   <xacro:arg name="stereo_camera_simulate_imu" default="true"/>
-  <!-- mount_arm:=true bolts the indomitus_arm onto main_body_link.-->
-  <xacro:arg name="mount_arm" default="false"/>
   <!-- Main robot description -->
   <xacro:include filename="$(find rover_description)/urdf/rover.urdf.xacro"/>
