Commit message: FEAT: restore navigation stack (#606)
- Restored ZED2i and EKF in `rover.launch.py`; new `zed2i_mode` argument (`rgb` / `nav` / `record`)
- Added a ZED2i `record` mode (`zed2i_record.yaml`) for traversability dataset recording
- Restored the `hw_ws` workspace in the Dockerfile (new `hw-builder` stage building sllidar and the ZED wrapper/description on Stereolabs CUDA images); CI, compose files and scripts adjusted
- Moved debugging tools from the Dockerfile into `indomitus_desktop/package.xml`
- Un-ignored `rover_localization`, `rover_navigation`, `rover_costmap_plugins` and removed them from the rsync deploy filter; `rover_aruco` still temporarily ignored
- EKF now fuses velocities from wheel and ZED2i odometry instead of absolute positions; sim config unified with the real one
- Fixed ZED2i/SLAM topic names and the sim spawner namespace broken by the rover namespace
- Fixed the TF lookup in the tilt broadcaster node
- Fixed RViz on Wayland (`QT_QPA_PLATFORM=xcb`)
- Updated ZED2i position in the URDF and configs
- Nav2: `default_server_timeout` increased to 1000, `xy_goal_tolerance` to 0.3
- Added `rosbag2_storage_mcap` and `rclcpp_components` dependencies; prod compose mounts a directory for ROS 2 bags
- Reworked `kill_node` alias (exact name matching, SIGINT → SIGTERM → SIGKILL escalation, check that the process stopped); added `launch_arm` alias

File: src/rover/rover_description/urdf/properties.xacro (robot description, xacro)
@@ -78,7 +78,7 @@
   <xacro:property name="zed2i_x" value="${body_length / 2.0 + 0.05}"/>
   <xacro:property name="zed2i_y" value="0.0"/>
-  <xacro:property name="zed2i_z" value="${body_height / 2.0 + 0.05}"/>
+  <xacro:property name="zed2i_z" value="${body_height / 2.0 - 0.07}"/>
   <xacro:property name="zed2i_rx" value="0.0"/>
-  <xacro:property name="zed2i_ry" value="${pi/12}"/>
+  <xacro:property name="zed2i_ry" value="${radians(37)}"/>
   <xacro:property name="zed2i_rz" value="0.0"/>
   <!-- ===================== LIDAR POSSITION ===================== -->

Commit message: chroe: more new tracks added; parameters tuned

File: src/rover/rover_description/urdf/properties.xacro (robot description, xacro)
@@ -76,5 +76,5 @@
   <xacro:property name="wheel_kd" value="1.0"/>
   <!-- ===================== ZED2I POSSITION ===================== -->
-  <xacro:property name="zed2i_x" value="${body_length / 2.0 + 0.05}"/>
+  <xacro:property name="zed2i_x" value="${body_length / 2.0 + 0.18}"/>
   <xacro:property name="zed2i_y" value="0.0"/>
   <xacro:property name="zed2i_z" value="${body_height / 2.0 - 0.07}"/>
